Commit message: savo_description partially done

File: savo_ws/src/shared/savo_description/urdf/materials.xacro (robot description, xacro)
@@ -1 +1,60 @@
-<!-- TODO: common colors/materials -->
+<?xml version="1.0"?>
+<robot xmlns:xacro="http://www.ros.org/wiki/xacro">
+  <material name="savo_black">
+    <color rgba="0.02 0.02 0.02 1.0"/>
+  </material>
+  <material name="savo_dark_gray">
+    <color rgba="0.12 0.12 0.12 1.0"/>
+  </material>
+  <material name="savo_gray">
+    <color rgba="0.35 0.35 0.35 1.0"/>
+  </material>
+  <material name="savo_light_gray">
+    <color rgba="0.70 0.70 0.70 1.0"/>
+  </material>
+  <material name="savo_white">
+    <color rgba="0.92 0.92 0.90 1.0"/>
+  </material>
+  <material name="savo_blue">
+    <color rgba="0.00 0.25 0.85 1.0"/>
+  </material>
+  <material name="savo_cyan">
+    <color rgba="0.00 0.75 0.95 1.0"/>
+  </material>
+  <material name="savo_green">
+    <color rgba="0.00 0.65 0.25 1.0"/>
+  </material>
+  <material name="savo_red">
+    <color rgba="0.85 0.05 0.05 1.0"/>
+  </material>
+  <material name="savo_orange">
+    <color rgba="1.00 0.45 0.05 1.0"/>
+  </material>
+  <material name="savo_yellow">
+    <color rgba="1.00 0.85 0.05 1.0"/>
+  </material>
+  <material name="savo_rubber">
+    <color rgba="0.01 0.01 0.01 1.0"/>
+  </material>
+  <material name="savo_lidar">
+    <color rgba="0.05 0.05 0.05 1.0"/>
+  </material>
+  <material name="savo_camera">
+    <color rgba="0.04 0.04 0.04 1.0"/>
+  </material>
+  <material name="savo_display">
+    <color rgba="0.00 0.00 0.00 1.0"/>
+  </material>
+  <material name="savo_pcb">
+    <color rgba="0.00 0.28 0.12 1.0"/>
+  </material>
+  <material name="savo_core_pi">
+    <color rgba="0.12 0.35 0.12 1.0"/>
+  </material>
+  <material name="savo_edge_pi">
+    <color rgba="0.12 0.22 0.45 1.0"/>
+  </material>
+  <material name="savo_transparent">
+    <color rgba="0.70 0.85 1.00 0.35"/>
+  </material>
+</robot>

File: savo_ws/src/shared/savo_description/urdf/robot_savo.urdf.xacro (robot description, xacro)
@@ -1 +1,31 @@
-<!-- TODO: robot physical model (Pi, LiDAR, wheels, etc.) -->
+<?xml version="1.0"?>
+<robot name="robot_savo" xmlns:xacro="http://www.ros.org/wiki/xacro">
+  <xacro:arg name="use_transmissions" default="false"/>
+  <xacro:arg name="use_gazebo" default="false"/>
+  <xacro:include filename="$(find savo_description)/urdf/materials.xacro"/>
+  <xacro:include filename="$(find savo_description)/urdf/macros/inertial_macro.xacro"/>
+  <xacro:include filename="$(find savo_description)/urdf/macros/box_macro.xacro"/>
+  <xacro:include filename="$(find savo_description)/urdf/macros/cylinder_macro.xacro"/>
+  <xacro:include filename="$(find savo_description)/urdf/macros/wheel_macro.xacro"/>
+  <xacro:include filename="$(find savo_description)/urdf/macros/sensor_macro.xacro"/>
+  <xacro:include filename="$(find savo_description)/urdf/macros/camera_macro.xacro"/>
+  <xacro:include filename="$(find savo_description)/urdf/macros/pi_mount_macro.xacro"/>
+  <xacro:include filename="$(find savo_description)/urdf/robot_savo_core.xacro"/>
+  <xacro:include filename="$(find savo_description)/urdf/robot_savo_wheels.xacro"/>
+  <xacro:include filename="$(find savo_description)/urdf/robot_savo_sensors.xacro"/>
+  <xacro:include filename="$(find savo_description)/urdf/robot_savo_two_pi.xacro"/>
+  <xacro:include filename="$(find savo_description)/urdf/robot_savo_costmap_frames.xacro"/>
+  <xacro:include filename="$(find savo_description)/urdf/robot_savo_transmissions.xacro"/>
+  <xacro:include filename="$(find savo_description)/urdf/robot_savo_gazebo.xacro"/>
+  <xacro:robot_savo_core/>
+  <xacro:robot_savo_wheels/>
+  <xacro:robot_savo_sensors/>
+  <xacro:robot_savo_two_pi/>
+  <xacro:robot_savo_costmap_frames/>
+  <xacro:if value="$(arg use_transmissions)">
+    <xacro:robot_savo_transmissions/>
+  </xacro:if>
+  <xacro:if value="$(arg use_gazebo)">
+    <xacro:robot_savo_gazebo/>
+  </xacro:if>
+</robot>
