Commit message: savo

File: savo_ws/src/shared/savo_description/urdf/robot_savo.urdf.xacro (robot description, xacro)
@@ -3,31 +3,33 @@
   <xacro:arg name="use_transmissions" default="false"/>
   <xacro:arg name="use_gazebo" default="false"/>
-  <xacro:arg name="base_length" default="0.330"/>
-  <xacro:arg name="base_width" default="0.240"/>
-  <xacro:arg name="base_height" default="0.060"/>
-  <xacro:arg name="base_link_z" default="0.065"/>
+  <xacro:arg name="base_length" default="0.2796"/>
+  <xacro:arg name="base_width" default="0.2100"/>
+  <xacro:arg name="base_height" default="0.0040"/>
+  <xacro:arg name="base_link_z" default="0.0325"/>
   <xacro:arg name="deck_thickness" default="0.004"/>
-  <xacro:arg name="deck_spacing" default="0.070"/>
+  <xacro:arg name="base_plate_z" default="-0.0185"/>
+  <xacro:arg name="first_plate_z" default="0.0475"/>
+  <xacro:arg name="second_plate_z" default="0.1675"/>
   <xacro:arg name="base_mass" default="1.20"/>
   <xacro:arg name="deck_mass" default="0.20"/>
   <xacro:arg name="wheel_radius" default="0.0325"/>
   <xacro:arg name="wheel_width" default="0.030"/>
-  <xacro:arg name="wheel_front_x" default="0.115"/>
-  <xacro:arg name="wheel_rear_x" default="-0.115"/>
-  <xacro:arg name="wheel_left_y" default="0.100"/>
-  <xacro:arg name="wheel_right_y" default="-0.100"/>
-  <xacro:arg name="wheel_z" default="-0.030"/>
+  <xacro:arg name="wheel_front_x" default="0.080"/>
+  <xacro:arg name="wheel_rear_x" default="-0.080"/>
+  <xacro:arg name="wheel_left_y" default="0.108"/>
+  <xacro:arg name="wheel_right_y" default="-0.108"/>
+  <xacro:arg name="wheel_z" default="0.0"/>
   <xacro:arg name="wheel_mass" default="0.12"/>
-  <xacro:arg name="lidar_xyz" default="0 0 0.205"/>
+  <xacro:arg name="lidar_xyz" default="0 0 0.2975"/>
   <xacro:arg name="lidar_rpy" default="0 0 0"/>
-  <xacro:arg name="imu_xyz" default="0 0 0.075"/>
+  <xacro:arg name="imu_xyz" default="0 -0.0465 -0.0175"/>
   <xacro:arg name="imu_rpy" default="0 0 0"/>
-  <xacro:arg name="camera_xyz" default="0.135 0 0.155"/>
+  <xacro:arg name="camera_xyz" default="0.130 0 0.1925"/>
   <xacro:arg name="camera_rpy" default="0 0 0"/>
-  <xacro:arg name="tof_left_xyz" default="0.125 0.090 0.070"/>
-  <xacro:arg name="tof_left_rpy" default="0 0 0"/>
-  <xacro:arg name="tof_right_xyz" default="0.125 -0.090 0.070"/>
-  <xacro:arg name="tof_right_rpy" default="0 0 0"/>
-  <xacro:arg name="ultrasonic_xyz" default="0.150 0 0.070"/>
+  <xacro:arg name="tof_left_xyz" default="0 0.106 -0.0075"/>
+  <xacro:arg name="tof_left_rpy" default="0 0 1.57079632679"/>
+  <xacro:arg name="tof_right_xyz" default="0 -0.106 -0.0075"/>
+  <xacro:arg name="tof_right_rpy" default="0 0 -1.57079632679"/>
+  <xacro:arg name="ultrasonic_xyz" default="0.137 0 0.0235"/>
   <xacro:arg name="ultrasonic_rpy" default="0 0 0"/>
   <xacro:arg name="display_xyz" default="0.115 0 0.145"/>
@@ -35,6 +37,7 @@
   <xacro:arg name="respeaker_xyz" default="0 0 0.180"/>
   <xacro:arg name="respeaker_rpy" default="0 0 0"/>
-  <xacro:arg name="pantilt_mount_xyz" default="0 0 0"/>
+  <xacro:arg name="pantilt_mount_xyz" default="0.115 0 0.2115"/>
   <xacro:arg name="pantilt_mount_rpy" default="0 0 0"/>
+  <xacro:arg name="depth_obstacle_xyz" default="0.130 0 0.1925"/>
   <xacro:include filename="$(find savo_description)/urdf/materials.xacro"/>
   <xacro:include filename="$(find savo_description)/urdf/macros/inertial_macro.xacro"/>
@@ -55,5 +58,8 @@
     base_length="$(arg base_length)" base_width="$(arg base_width)"
     base_height="$(arg base_height)" base_link_z="$(arg base_link_z)"
-    deck_thickness="$(arg deck_thickness)" deck_spacing="$(arg deck_spacing)"
+    deck_thickness="$(arg deck_thickness)"
+    base_plate_z="$(arg base_plate_z)"
+    first_plate_z="$(arg first_plate_z)"
+    second_plate_z="$(arg second_plate_z)"
     base_mass="$(arg base_mass)" deck_mass="$(arg deck_mass)"/>
   <xacro:robot_savo_wheels
@@ -74,5 +80,5 @@
     pantilt_mount_rpy="$(arg pantilt_mount_rpy)"/>
   <xacro:robot_savo_two_pi/>
-  <xacro:robot_savo_costmap_frames/>
+  <xacro:robot_savo_costmap_frames depth_obstacle_xyz="$(arg depth_obstacle_xyz)"/>
   <xacro:if value="$(arg use_transmissions)">
     <xacro:robot_savo_transmissions/>

File: savo_ws/src/shared/savo_description/urdf/robot_savo_core.xacro (robot description, xacro)
@@ -3,10 +3,12 @@
   <xacro:macro name="robot_savo_core"
     params="
-      base_length:=0.330
-      base_width:=0.240
-      base_height:=0.060
-      base_link_z:=0.065
+      base_length:=0.2796
+      base_width:=0.2100
+      base_height:=0.0040
+      base_link_z:=0.0325
       deck_thickness:=0.004
-      deck_spacing:=0.070
+      base_plate_z:=-0.0185
+      first_plate_z:=0.0475
+      second_plate_z:=0.1675
       base_mass:=1.20
       deck_mass:=0.20
@@ -33,5 +35,5 @@
       name="chassis_link"
       parent="base_link"
-      xyz="0 0 0"
+      xyz="0 0 ${base_plate_z}"
       rpy="0 0 0"
       size_xyz="${base_length} ${base_width} ${base_height}"
@@ -40,18 +42,9 @@
     />
     <xacro:fixed_box
-      name="lower_deck_link"
+      name="middle_deck_link"
       parent="base_link"
-      xyz="0 0 ${base_height / 2.0 + deck_thickness / 2.0}"
+      xyz="0 0 ${first_plate_z}"
       rpy="0 0 0"
       size_xyz="${base_length} ${base_width} ${deck_thickness}"
-      mass="${deck_mass}"
-      material="savo_black"
-    />
-    <xacro:fixed_box
-      name="middle_deck_link"
-      parent="base_link"
-      xyz="0 0 ${base_height / 2.0 + deck_spacing}"
-      rpy="0 0 0"
-      size_xyz="${base_length * 0.92} ${base_width * 0.92} ${deck_thickness}"
       mass="${deck_mass}"
       material="savo_gray"
@@ -60,7 +53,7 @@
       name="top_deck_link"
       parent="base_link"
-      xyz="0 0 ${base_height / 2.0 + deck_spacing * 2.0}"
+      xyz="0 0 ${second_plate_z}"
       rpy="0 0 0"
-      size_xyz="${base_length * 0.82} ${base_width * 0.82} ${deck_thickness}"
+      size_xyz="${base_length} ${base_width} ${deck_thickness}"
       mass="${deck_mass}"
       material="savo_light_gray"

File: savo_ws/src/shared/savo_description/urdf/robot_savo_costmap_frames.xacro (robot description, xacro)
@@ -4,6 +4,5 @@
     params="
       parent:=base_link
-      depth_obstacle_x:=0.135
-      depth_obstacle_z:=0.155
+      depth_obstacle_xyz:='0.130 0 0.1925'
       local_costmap_z:=0.000
       footprint_z:=0.000
@@ -13,5 +12,5 @@
       <parent link="${parent}"/>
       <child link="depth_obstacle_frame"/>
-      <origin xyz="${depth_obstacle_x} 0 ${depth_obstacle_z}" rpy="0 0 0"/>
+      <origin xyz="${depth_obstacle_xyz}" rpy="0 0 0"/>
     </joint>
     <link name="local_costmap_frame"/>

File: savo_ws/src/shared/savo_description/urdf/robot_savo_gazebo.xacro (robot description, xacro)
@@ -4,7 +4,4 @@
     <gazebo reference="chassis_link">
       <material>Gazebo/DarkGrey</material>
-    </gazebo>
-    <gazebo reference="lower_deck_link">
-      <material>Gazebo/Black</material>
     </gazebo>
     <gazebo reference="middle_deck_link">

File: savo_ws/src/shared/savo_description/urdf/robot_savo_sensors.xacro (robot description, xacro)
@@ -4,13 +4,13 @@
     params="
       parent:=base_link
-      lidar_xyz:='0 0 0.205' lidar_rpy:='0 0 0'
-      imu_xyz:='0 0 0.075' imu_rpy:='0 0 0'
-      camera_xyz:='0.135 0 0.155' camera_rpy:='0 0 0'
-      tof_left_xyz:='0.125 0.090 0.070' tof_left_rpy:='0 0 0'
-      tof_right_xyz:='0.125 -0.090 0.070' tof_right_rpy:='0 0 0'
-      ultrasonic_xyz:='0.150 0 0.070' ultrasonic_rpy:='0 0 0'
+      lidar_xyz:='0 0 0.2975' lidar_rpy:='0 0 0'
+      imu_xyz:='0 -0.0465 -0.0175' imu_rpy:='0 0 0'
+      camera_xyz:='0.130 0 0.1925' camera_rpy:='0 0 0'
+      tof_left_xyz:='0 0.106 -0.0075' tof_left_rpy:='0 0 1.57079632679'
+      tof_right_xyz:='0 -0.106 -0.0075' tof_right_rpy:='0 0 -1.57079632679'
+      ultrasonic_xyz:='0.137 0 0.0235' ultrasonic_rpy:='0 0 0'
       display_xyz:='0.115 0 0.145' display_rpy:='0 0 0'
       respeaker_xyz:='0 0 0.180' respeaker_rpy:='0 0 0'
-      pantilt_mount_xyz:='0 0 0' pantilt_mount_rpy:='0 0 0'
+      pantilt_mount_xyz:='0.115 0 0.2115' pantilt_mount_rpy:='0 0 0'
     ">
     <xacro:sensor_cylinder

File: savo_ws/src/shared/savo_description/urdf/robot_savo_wheels.xacro (robot description, xacro)
@@ -6,9 +6,9 @@
       wheel_radius:=0.0325
       wheel_width:=0.030
-      wheel_front_x:=0.115
-      wheel_rear_x:=-0.115
-      wheel_left_y:=0.100
-      wheel_right_y:=-0.100
-      wheel_z:=-0.030
+      wheel_front_x:=0.080
+      wheel_rear_x:=-0.080
+      wheel_left_y:=0.108
+      wheel_right_y:=-0.108
+      wheel_z:=0.0
       wheel_mass:=0.12
     ">

Commit message: savo

File: savo_ws/src/shared/savo_description/urdf/robot_savo.urdf.xacro (robot description, xacro)
@@ -6,9 +6,13 @@
   <xacro:arg name="base_width" default="0.2100"/>
   <xacro:arg name="base_height" default="0.0040"/>
+  <xacro:arg name="third_plate_length" default="0.1420"/>
+  <xacro:arg name="third_plate_width" default="0.1440"/>
+  <xacro:arg name="third_plate_height" default="0.0040"/>
   <xacro:arg name="base_link_z" default="0.0325"/>
   <xacro:arg name="deck_thickness" default="0.004"/>
-  <xacro:arg name="base_plate_z" default="-0.0185"/>
+  <xacro:arg name="base_plate_z" default="-0.0175"/>
   <xacro:arg name="first_plate_z" default="0.0475"/>
-  <xacro:arg name="second_plate_z" default="0.1675"/>
+  <xacro:arg name="second_plate_z" default="0.1635"/>
+  <xacro:arg name="third_plate_z" default="0.2475"/>
   <xacro:arg name="base_mass" default="1.20"/>
   <xacro:arg name="deck_mass" default="0.20"/>
@@ -58,8 +62,12 @@
     base_length="$(arg base_length)" base_width="$(arg base_width)"
     base_height="$(arg base_height)" base_link_z="$(arg base_link_z)"
+    third_plate_length="$(arg third_plate_length)"
+    third_plate_width="$(arg third_plate_width)"
+    third_plate_height="$(arg third_plate_height)"
     deck_thickness="$(arg deck_thickness)"
     base_plate_z="$(arg base_plate_z)"
     first_plate_z="$(arg first_plate_z)"
     second_plate_z="$(arg second_plate_z)"
+    third_plate_z="$(arg third_plate_z)"
     base_mass="$(arg base_mass)" deck_mass="$(arg deck_mass)"/>
   <xacro:robot_savo_wheels

File: savo_ws/src/shared/savo_description/urdf/robot_savo_core.xacro (robot description, xacro)
@@ -6,9 +6,13 @@
       base_width:=0.2100
       base_height:=0.0040
+      third_plate_length:=0.1420
+      third_plate_width:=0.1440
+      third_plate_height:=0.0040
       base_link_z:=0.0325
       deck_thickness:=0.004
-      base_plate_z:=-0.0185
+      base_plate_z:=-0.0175
       first_plate_z:=0.0475
-      second_plate_z:=0.1675
+      second_plate_z:=0.1635
+      third_plate_z:=0.2475
       base_mass:=1.20
       deck_mass:=0.20
@@ -59,4 +63,13 @@
       material="savo_light_gray"
     />
+    <xacro:fixed_box
+      name="lidar_deck_link"
+      parent="base_link"
+      xyz="0 0 ${third_plate_z}"
+      rpy="0 0 0"
+      size_xyz="${third_plate_length} ${third_plate_width} ${third_plate_height}"
+      mass="${deck_mass}"
+      material="savo_light_gray"
+    />
   </xacro:macro>
 </robot>

File: savo_ws/src/shared/savo_description/urdf/robot_savo_gazebo.xacro (robot description, xacro)
@@ -9,4 +9,7 @@
     </gazebo>
     <gazebo reference="top_deck_link">
+      <material>Gazebo/White</material>
+    </gazebo>
+    <gazebo reference="lidar_deck_link">
       <material>Gazebo/White</material>
     </gazebo>
