Commit message: Lock Robot Savo production geometry

File: savo_ws/src/shared/savo_description/urdf/macros/camera_macro.xacro (robot description, xacro)
@@ -12,5 +12,5 @@
     />
   </xacro:macro>
-  <xacro:macro name="camera_frames" params="name parent xyz rpy">
+  <xacro:macro name="camera_frames" params="name parent xyz rpy color_xyz color_rpy">
     <link name="${name}_link"/>
     <joint name="${name}_joint" type="fixed">
@@ -23,5 +23,5 @@
       <parent link="${name}_link"/>
       <child link="${name}_color_frame"/>
-      <origin xyz="0 0 0" rpy="0 0 0"/>
+      <origin xyz="${color_xyz}" rpy="${color_rpy}"/>
     </joint>
     <link name="${name}_color_optical_frame"/>
@@ -44,5 +44,5 @@
     </joint>
   </xacro:macro>
-  <xacro:macro name="depth_camera" params="name parent xyz rpy size_xyz mass material">
+  <xacro:macro name="depth_camera" params="name parent xyz rpy color_xyz color_rpy size_xyz mass material">
     <xacro:camera_body
       name="${name}_body"
@@ -59,4 +59,6 @@
       xyz="0 0 0"
       rpy="0 0 0"
+      color_xyz="${color_xyz}"
+      color_rpy="${color_rpy}"
     />
   </xacro:macro>

File: savo_ws/src/shared/savo_description/urdf/robot_savo.urdf.xacro (robot description, xacro)
@@ -11,8 +11,8 @@
   <xacro:arg name="base_link_z" default="0.0325"/>
   <xacro:arg name="deck_thickness" default="0.004"/>
-  <xacro:arg name="base_plate_z" default="-0.0175"/>
-  <xacro:arg name="first_plate_z" default="0.0475"/>
-  <xacro:arg name="second_plate_z" default="0.1635"/>
-  <xacro:arg name="third_plate_z" default="0.2475"/>
+  <xacro:arg name="base_plate_z" default="-0.0155"/>
+  <xacro:arg name="first_plate_z" default="0.0495"/>
+  <xacro:arg name="second_plate_z" default="0.1655"/>
+  <xacro:arg name="third_plate_z" default="0.2495"/>
   <xacro:arg name="base_mass" default="1.20"/>
   <xacro:arg name="deck_mass" default="0.20"/>
@@ -31,4 +31,6 @@
   <xacro:arg name="camera_xyz" default="0.130 0 0.1925"/>
   <xacro:arg name="camera_rpy" default="0 0 0"/>
+  <xacro:arg name="camera_color_xyz" default="-0.000287127564661 0.014867129735649 0.000134048212203"/>
+  <xacro:arg name="camera_color_rpy" default="-0.007168423593435 0.000448528015039 0.010917321307075"/>
   <xacro:arg name="tof_left_xyz" default="0 0.106 -0.0075"/>
   <xacro:arg name="tof_left_rpy" default="0 0 1.57079632679"/>
@@ -80,4 +82,6 @@
     imu_xyz="$(arg imu_xyz)" imu_rpy="$(arg imu_rpy)"
     camera_xyz="$(arg camera_xyz)" camera_rpy="$(arg camera_rpy)"
+    camera_color_xyz="$(arg camera_color_xyz)"
+    camera_color_rpy="$(arg camera_color_rpy)"
     tof_left_xyz="$(arg tof_left_xyz)" tof_left_rpy="$(arg tof_left_rpy)"
     tof_right_xyz="$(arg tof_right_xyz)" tof_right_rpy="$(arg tof_right_rpy)"

File: savo_ws/src/shared/savo_description/urdf/robot_savo_core.xacro (robot description, xacro)
@@ -11,8 +11,8 @@
       base_link_z:=0.0325
       deck_thickness:=0.004
-      base_plate_z:=-0.0175
-      first_plate_z:=0.0475
-      second_plate_z:=0.1635
-      third_plate_z:=0.2475
+      base_plate_z:=-0.0155
+      first_plate_z:=0.0495
+      second_plate_z:=0.1655
+      third_plate_z:=0.2495
       base_mass:=1.20
       deck_mass:=0.20

File: savo_ws/src/shared/savo_description/urdf/robot_savo_sensors.xacro (robot description, xacro)
@@ -7,4 +7,6 @@
       imu_xyz:='0 -0.0465 -0.0175' imu_rpy:='0 0 0'
       camera_xyz:='0.130 0 0.1925' camera_rpy:='0 0 0'
+      camera_color_xyz:='-0.000287127564661 0.014867129735649 0.000134048212203'
+      camera_color_rpy:='-0.007168423593435 0.000448528015039 0.010917321307075'
       tof_left_xyz:='0 0.106 -0.0075' tof_left_rpy:='0 0 1.57079632679'
       tof_right_xyz:='0 -0.106 -0.0075' tof_right_rpy:='0 0 -1.57079632679'
@@ -39,4 +41,6 @@
       xyz="${camera_xyz}"
       rpy="${camera_rpy}"
+      color_xyz="${camera_color_xyz}"
+      color_rpy="${camera_color_rpy}"
       size_xyz="0.090 0.025 0.025"
       mass="0.075"
